Commit message: Sim saatini, kamera goru s acisini ve bridge kurulumunu duzelt
Gazebo tarafinda tespit edilen ve uzerinde anlasilan sorunlar:

- /clock koprulenmiyordu ve hicbir node use_sim_time kullanmiyordu;
  Gazebo sim-time damgali mesaj yayinlarken ROS node'lari wall-clock
  kullaniyordu. Simdilik sadece static TF kullanildigi icin fark
  edilmemisti, ama EKF devreye girdiginde TF lookup'lari kirilacakti.
  parameter_bridge'e use_sim_time BILEREK verilmiyor: /clock'u bizzat
  o yayinladigi icin kendi saatini beklemesi kilitlenmeye yol acar.

- Kamera duz bakiyordu; tag'ler z=1.2 m'de, kamera z=0.12 m'de oldugu
  icin tag ancak 2.39 m'den uzakta kadraja sigiyordu. 15 derece yukari
  pitch bu sinirii 1.34 m'ye indiriyor ve tipik 3.84 m calisma
  mesafesinde tag'i optik eksene oturtuyor.

- JointStatePublisher plugin'i veri yayinliyordu ama /joint_states
  koprulenmedigi icin robot_state_publisher eklem acisi alamiyor,
  direksiyon/tekerlek TF'lerini yayinlayamiyordu.

- Bridge'de her topic cift yonlu (@) tanimliydi; artik her biri
  gercekten ihtiyac duyulan tek yonde ([ ya da ]).

- Script'lerdeki sabit sandbox yollari (/workspace/...) script'in kendi
  konumundan turetiliyor.

- robot_state.sh car.urdf'i sadece yoksa uretiyordu, bu yuzden xacro'da
  yapilan degisiklik eski ciktiyla sessizce goz ardi ediliyordu.

Lidar menzili, lidar montaj yuksekligi ve tag pose'lari bilerek
degistirilmedi.

Co-Authored-By: Claude Opus 5 <noreply@anthropic.com>

File: gazebo-env/urdf/car.urdf.xacro (robot description, xacro)
@@ -134,4 +134,18 @@
   <xacro:property name="camera_origin_x"  value="${chassis_length/2}"/>
   <xacro:property name="camera_origin_z"  value="${wheel_radius + chassis_height*0.7}"/>
+  <!-- camera_pitch: kamerayi YUKARI egen aci (radyan). Tag'ler duvarda
+       z=1.2 m'de, kamera ise z=0.12 m'de; aradaki 1.08 m'lik fark
+       yuzunden duz bakan bir kamera tag'i ancak 2.39 m'den UZAKTAN
+       kadraja sigdirabiliyordu (daha yakinda tag kadrajin ustunden
+       tasiyordu). 15 derece yukari pitch ile bu sinir 1.34 m'ye
+       iniyor; ayrica oda merkezinden duvara olan 3.84 m'lik tipik
+       calisma mesafesinde tag neredeyse tam optik eksene oturuyor
+       (+0.7 derece), bu da PnP pose kestiriminde lens kenarindaki
+       bozulmadan kacinmayi sagliyor.
+       DIKKAT: ROS/REP-103 konvansiyonunda pitch +y ekseni etrafinda
+       doner ve POZITIF pitch burnu ASAGI eger. Bu yuzden asagidaki
+       camera_joint'te isaret NEGATIF kullaniliyor. -->
+  <xacro:property name="camera_pitch"     value="0.2618"/> <!-- 15 derece -->
+  <xacro:property name="camera_joint_pitch" value="${-camera_pitch}"/>
   <!-- OPERASYONEL:
        - camera_horizontal_fov: yatay gorus acisi (radyan). Genis FOV
@@ -434,5 +448,5 @@
     <parent link="base_link"/>
     <child link="camera_link"/>
-    <origin xyz="${camera_origin_x} 0 ${camera_origin_z}" rpy="0 0 0"/>
+    <origin xyz="${camera_origin_x} 0 ${camera_origin_z}" rpy="0 ${camera_joint_pitch} 0"/>
   </joint>
   <link name="camera_link_optical"/>
